File: STM32_PCB_design/STM32_PCB_design.kicad_sch (KiCad schematic)
At the start: 10 parts

Commit message: STM32 configuration pins
Parts:
- added C?: 100n, symbol Device:C
- added R?: 10k, symbol Device:R
- added SW?: SW_SPDT, symbol Switch:SW_SPDT
Connections:
- net +3.3V: now also SW?.3 (C)
- net GND: now also C?.2, SW?.1 (A)
- net BOOT0: now reaches U?.44 (BOOT0)
- net BOOT0: now also R?.2
- net NRST: now reaches U?.7 (NRST)
- net NRST: now also C?.1
- new net SW_BOOT0: R?.1, SW?.2 (B)
Other:
- note added: "By default,mcu runs without going to booloader mode"
- note added: "Pins Description: NSRT -> if is pulled low this will put this microcontroller into reset mode. Tipically is put high. BOOT0 -> Enables or disables internal bootloader esp32. The way to programming one of these is via JTAG or Serial wired debug. If we put pin high, this enables interfaces such as uart or usb or others."
